File: PCB/falcon-core.kicad_pcb (KiCad board)
At the start: 4 copper layers, 32 x 46 mm, 89 parts, among them J2 USB_C_Receptacle_USB2.0_16P, J3 Conn_01x04_Socket, J4 Conn_01x04_Socket, Q1 AO3401A, SW1 SW_SPDT, U1 ESP32-S3-WROOM-1, U10 ME6211C28M5, U11 BMI270, U13 VL53L5CXV0GC_1, U15 MMC5633NJL, U2 DRV8212P, U3 DRV8212P, U4 DRV8212P, U5 DRV8212P, U6 TPS63001, U7 TP4057, U8 ME6211C28M5, U9 ME6211C12M5

Commit message: add first round of software
Parts:
- added C30: 100nF, PCM_JLCPCB:C_0402, F.Cu at (8.20, 15.7)
- added C31: 100nF, PCM_JLCPCB:C_0402, F.Cu at (19.6, 13.8)
- added C36: 100nF, PCM_JLCPCB:C_0402, F.Cu at (8.60, 37.4)
- added S1: Tactile Button, 160gf, PCM_JLCPCB:SW_TS-1088-AR02016, F.Cu at (21.2, 28.3)
- added S2: Tactile Button, 160gf, PCM_JLCPCB:SW_TS-1088-AR02016, F.Cu at (21.1, 20.1)
- moved SW1 1.55 mm to (3.80, 9.75)
- moved C1 1.20 mm to (7.70, 9.25)
- moved C2 1.20 mm to (7.70, 14.2)
- moved R19 1.20 mm to (9.07, 15.1)
- moved U8 1.20 mm to (8.20, 11.8)
- moved C3 0.60 mm to (11.6, 14.2)
- moved C4 0.60 mm to (11.6, 9.25)
- moved U1 0.60 mm to (6.15, 27.2)
- moved U9 0.60 mm to (12.1, 11.8)
- moved D3 0.55 mm to (10.2, 37.4)
- moved C21 0.54 mm to (23.3, 25.7)
- moved C22 0.51 mm to (23.2, 20.5)
- moved R11 0.50 mm to (18.2, 38.0)
- moved R20 0.35 mm to (19.8, 16.1)
- moved R18 0.30 mm to (20.5, 13.8)
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Connections:
- net Net-(U1-EN) renamed /EN
- net Net-(U1-IO0) renamed /BOOT
- FPC1 pad 17: +3V3 -> GND
- FPC1 pad 19: GND -> +3V3
- TP4 pad 1: +3V3 -> unconnected-(TP4-Pad1)
- U1 pad 8: /M4_IN1 -> /M4_IN2
- U1 pad 9: /M4_IN2 -> /M4_IN1
Routing:
- net /EN: track 22.4 -> 47.0 mm, vias 2 -> 4
- net GND: track 46.9 -> 51.5 mm, vias 56 -> 74
- net /BOOT: track 17.0 -> 20.0 mm, vias 2 -> 3
- net /BAT_ADC: track 31.4 -> 33.3 mm
- net +2V8A: track 10.0 -> 8.34 mm
- net Net-(Q1-G): track 29.8 -> 28.5 mm
- net /M3_IN1: track 37.2 -> 38.3 mm
- net +3V3: track 71.2 -> 70.1 mm
- net /SCL: track 35.2 -> 34.1 mm
- net /SIOC: track 24.5 -> 23.4 mm
- net /SIOD: track 24.4 -> 23.4 mm
- net /M4_IN2: track 27.8 -> 28.8 mm
- net /M1_IN2: track 31.3 -> 32.1 mm
- net /M4_IN1: track 28.5 -> 27.7 mm
- net /M3_IN2: track 38.8 -> 39.5 mm
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- added copper zone on In2.Cu, net GND
Other:
- board text added: "BOOT"
- board text added: "EN"
- board text added: "V1.1"

Commit message: Refactor code structure for improved readability and maintainability
Parts:
- U15: value MMC5633NJL -> MMC5603NJL
Connections:
- TP4 pad 1: unconnected-(TP4-Pad1) -> +3V3
