File: PCB/falcon-core.kicad_sch (KiCad schematic)
At the start: 89 parts, among them J2 USB_C_Receptacle_USB2.0_16P, J3 Conn_01x04_Socket, J4 Conn_01x04_Socket, Q1 AO3401A, SW1 SW_SPDT, U1 ESP32-S3-WROOM-1, U10 ME6211C28M5, U11 BMI270, U13 VL53L5CXV0GC_1, U15 MMC5633NJL, U2 DRV8212P, U3 DRV8212P, U4 DRV8212P, U5 DRV8212P, U6 TPS63001, U7 TP4057, U8 ME6211C28M5, U9 ME6211C12M5

Commit message: add first round of software
Parts:
- added C30, C31, C36: 100nF, PCM_JLCPCB:C_0402, symbol PCM_JLCPCB-Capacitors:0402,100nF
- added S1, S2: Tactile Button, 160gf, PCM_JLCPCB:SW_TS-1088-AR02016, symbol PCM_JLCPCB-Connectors_Buttons:Tactile Button, 160gf, 12V, 50mA, 4.0mm
- BAT1: LCSC (none) -> C23397052
- J3, J4: LCSC (none) -> C46061768
Connections:
- net +3V3: now also FPC1.19; no longer FPC1.17, TP4.1
- net BAT_ADC: now also C36.1
- net GND: now also FPC1.17, C30.2, C31.2, C36.2, S1.2 (B), S2.2 (B); no longer FPC1.19
- net M4_IN1: now also U1.9 (IO16); no longer U1.8 (IO15)
- net M4_IN2: now also U1.8 (IO15); no longer U1.9 (IO16)
- net EN: now reaches R19.1, TP1.1, U1.3 (EN)
- net EN: now also C30.1, S1.1 (A)
- net BOOT: now reaches R18.1, TP2.1, U1.27 (IO0)
- net BOOT: now also C31.1, S2.1 (A)
Other:
- moved on the sheet: FPC1, R18, R19

Commit message: Refactor code structure for improved readability and maintainability
Parts:
- U15: value MMC5633NJL -> MMC5603NJL; LCSC C3716174 -> C404328
Connections:
- net +3V3: now also TP4.1
Other:
- moved on the sheet: TP4
Changed lines of the file:
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@@
 	(symbol
 		(lib_id "Connector:TestPoint")
-		(at 30.48 87.63 90)
+		(at 62.23 75.565 270)
 		(unit 1)
 		(body_style 1)
@@
 		(fields_autoplaced yes)
 		(property "Reference" "TP4"
-			(at 27.178 81.915 90)
+			(at 67.31 74.2949 90)
 			(show_name no)
 			(do_not_autoplace no)
@@
 					(size 1.27 1.27)
 				)
+				(justify left)
 			)
 		)
 		(property "Value" "3V3"
-			(at 27.178 84.455 90)
+			(at 67.31 76.8349 90)
 			(show_name no)
 			(do_not_autoplace no)
@@
 					(size 1.27 1.27)
 				)
+				(justify left)
 			)
 		)
 		(property "Footprint" "TestPoint:TestPoint_Pad_D2.0mm"
-			(at 30.48 82.55 0)
+			(at 62.23 80.645 0)
 			(hide yes)
 			(show_name no)
@@
 		)
 		(property "Datasheet" ""
-			(at 30.48 82.55 0)
+			(at 62.23 80.645 0)
 			(show_name no)
 			(do_not_autoplace no)
@@
 		)
 		(property "Description" "test point"
-			(at 30.48 87.63 0)
+			(at 62.23 75.565 0)
 			(hide yes)
 			(show_name no)
@@
 			)
 		)
-		(property "Value" "MMC5633NJL"
+		(property "Value" "MMC5603NJL"
 			(at 151.765 190.4999 0)
 			(show_name no)
@@
 			)
 		)
-		(property "LCSC" "C3716174"
+		(property "LCSC" "C404328"
 			(at 160.02 200.66 0)
 			(hide yes)
